File: board/AudioBox.sch (KiCad schematic (older format))
At the start: 88 parts, among them J1 Conn_01x04_Male, J2 Conn_Coaxial_Power, J3 AudioJack3_SwitchT, J4 Conn_02x20_Odd_Even, U1 AD1938, U10 LDLN030, U2 TS912, U3 TS912, U4 TS912, U5 TS912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

Commit message: half placement done
Parts:
- removed J1: Conn_01x04_Male, Connector_PinHeader_2.54mm:PinHeader_1x04_P2.54mm_Vertical, symbol Connector:Conn_01x04_Male
- removed J2: Conn_Coaxial_Power, Connector_BarrelJack:BarrelJack_Wuerth_6941xx301002, symbol Connector_Generic:Conn_01x03
- removed R7: 100K, Resistor_SMD:R_0603_1608Metric_Pad1.05x0.95mm_HandSolder, symbol Device:R
- C12: value 10u -> 22u; PN GRM188R61E106KA73D -> GRM21BR61A226ME51L; Tolerance 10% -> 20%; Voltage 25V -> 10V
- R14, R15, R16, R17: Manufacturer Vishay Dale -> Yageo; PN CRCW0201100RFKED -> RC0603FR-07100RL
- R3: value 4.7K -> 2.2K; PN CRCW06034K70JNEAC -> CRCW06032K20FKEA
Connections:
- net +5VA is gone; now on net +5V: C27.2, U10.1 (IN), U10.3 (EN)
- net ADC_CM: now also U3.3 (+); no longer R3.2
- net IN_1: now also C12.2; no longer C12.1
- net at C20.1, R10.2, R8.1: now also U3.7; no longer U3.1
- net at R3.1, R8.2: now also U3.6 (-); no longer U3.2 (-)
- net at R10.1, R12.2: now also U3.2 (-); no longer U3.6 (-)
- net at C19.2, R12.1: now also U3.1; no longer U3.7
- net at C22.1, R11.2, R9.1: now also U4.7; no longer U4.1
- net at R4.1, R9.2: now also U4.6 (-); no longer U4.2 (-)
- net at R11.1, R13.2: now also U4.2 (-); no longer U4.6 (-)
- net at C21.1, R13.1: now also U4.1; no longer U4.7
- new net: C12.1, R3.2
Other:
- moved on the sheet: C1, C10, C18, C19, C2, C20, C23, C24, C27, C28, C29, C3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

Commit message: modified resistor values of the input buffer
Parts:
- IN1, IN2, OUT1, OUT2: symbol Audio:4833.222 -> AudioBox-rescue:4833.222-Audio
- J3: symbol Connector:AudioJack3_SwitchT -> AudioBox-rescue:AudioJack3_SwitchT-Connector
- R10, R13: value 4.7K -> 100K; PN CRCW06034K70JNEAC -> CRCW0603100KJNEAC; Tolerance 1% -> 5 %
- R11, R12, R8, R9: value 4.7K -> 100K; PN CRCW06034K70JNEAC -> CRCW0603100KJNEAC; Tolerance 1% -> 5%
- R3: value 2.2K -> 100K; PN CRCW06032K20FKEA -> CRCW0603100KJNEAC; Tolerance 1% -> 5
- R4: value 2.2K -> 100K; PN CRCW06032K20FKEA -> CRCW0603100KJNEAC; Tolerance 1% -> 5%
- U1: symbol Analog:AD1938 -> AudioBox-rescue:AD1938-Analog
- U10: symbol Regulator_Linear:LDLN030 -> AudioBox-rescue:LDLN030-Regulator_Linear
Changed lines of the file:
@@
 Connection ~ 2500 1350
 $Comp
-L Analog:AD1938 U1
+L AudioBox-rescue:AD1938-Analog U1
 U 1 1 5EBC8C13
 P 4800 5750
@@
 P 12400 3300
 F 0 "R9" V 12300 3200 50  0000 L CNN
-F 1 "4.7K" V 12500 3200 50  0000 L CNN
+F 1 "100K" V 12500 3200 50  0000 L CNN
 F 2 "Resistor_SMD:R_0603_1608Metric_Pad1.05x0.95mm_HandSolder" V 12330 3300 50  0001 C CNN
 F 3 "~" H 12400 3300 50  0001 C CNN
@@
 F 5 "" H 12400 3300 50  0001 C CNN "Material"
 F 6 "" H 12400 3300 50  0001 C CNN "Power"
-F 7 "1%" H 12400 3300 50  0001 C CNN "Tolerance"
+F 7 "5%" H 12400 3300 50  0001 C CNN "Tolerance"
 F 8 "Vishay Dale" H 12400 3300 50  0001 C CNN "Manufacturer"
-F 9 "	CRCW06034K70JNEAC" H 12400 3300 50  0001 C CNN "PN"
+F 9 "CRCW0603100KJNEAC" H 12400 3300 50  0001 C CNN "PN"
 	1    12400 3300
 	0    1    1    0
@@
 P 11650 3050
 F 0 "R4" V 11750 2950 50  0000 L CNN
-F 1 "2.2K" V 11850 2950 50  0000 L CNN
+F 1 "100K" V 11850 2950 50  0000 L CNN
 F 2 "Resistor_SMD:R_0603_1608Metric_Pad1.05x0.95mm_HandSolder" V 11580 3050 50  0001 C CNN
 F 3 "~" H 11650 3050 50  0001 C CNN
@@
 F 5 "" H 11650 3050 50  0001 C CNN "Material"
 F 6 "" H 11650 3050 50  0001 C CNN "Power"
-F 7 "1%" H 11650 3050 50  0001 C CNN "Tolerance"
+F 7 "5%" H 11650 3050 50  0001 C CNN "Tolerance"
 F 8 "Vishay Dale" H 11650 3050 50  0001 C CNN "Manufacturer"
-F 9 "CRCW06032K20FKEA" H 11650 3050 50  0001 C CNN "PN"
+F 9 "CRCW0603100KJNEAC" H 11650 3050 50  0001 C CNN "PN"
 	1    11650 3050
 	0    1    1    0
@@
 P 12900 1350
 F 0 "R10" V 12800 1250 50  0000 L CNN
-F 1 "4.7K" V 13000 1250 50  0000 L CNN
+F 1 "100K" V 13000 1250 50  0000 L CNN
 F 2 "Resistor_SMD:R_0603_1608Metric_Pad1.05x0.95mm_HandSolder" V 12830 1350 50  0001 C CNN
 F 3 "~" H 12900 1350 50  0001 C CNN
@@
 F 5 "" H 12900 1350 50  0001 C CNN "Material"
 F 6 "" H 12900 1350 50  0001 C CNN "Power"
-F 7 "1%" H 12900 1350 50  0001 C CNN "Tolerance"
+F 7 "5 %" H 12900 1350 50  0001 C CNN "Tolerance"
 F 8 "Vishay Dale" H 12900 1350 50  0001 C CNN "Manufacturer"
-F 9 "	CRCW06034K70JNEAC" H 12900 1350 50  0001 C CNN "PN"
+F 9 "CRCW0603100KJNEAC" H 12900 1350 50  0001 C CNN "PN"
 	1    12900 1350
 	0    1    1    0
@@
 P 13500 1700
 F 0 "R12" V 13300 1600 50  0000 L CNN
-F 1 "4.7K" V 13400 1600 50  0000 L CNN
+F 1 "100K" V 13400 1600 50  0000 L CNN
 F 2 "Resistor_SMD:R_0603_1608Metric_Pad1.05x0.95mm_HandSolder" V 13430 1700 50  0001 C CNN
 F 3 "~" H 13500 1700 50  0001 C CNN
@@
 F 5 "" H 13500 1700 50  0001 C CNN "Material"
 F 6 "" H 13500 1700 50  0001 C CNN "Power"
-F 7 "1%" H 13500 1700 50  0001 C CNN "Tolerance"
+F 7 "5%" H 13500 1700 50  0001 C CNN "Tolerance"
 F 8 "Vishay Dale" H 13500 1700 50  0001 C CNN "Manufacturer"
-F 9 "	CRCW06034K70JNEAC" H 13500 1700 50  0001 C CNN "PN"
+F 9 "CRCW0603100KJNEAC" H 13500 1700 50  0001 C CNN "PN"
 	1    13500 1700
 	0    1    1    0
@@
 P 12900 2950
 F 0 "R11" V 12800 2850 50  0000 L CNN
-F 1 "4.7K" V 13000 2850 50  0000 L CNN
+F 1 "100K" V 13000 2850 50  0000 L CNN
 F 2 "Resistor_SMD:R_0603_1608Metric_Pad1.05x0.95mm_HandSolder" V 12830 2950 50  0001 C CNN
 F 3 "~" H 12900 2950 50  0001 C CNN
@@
 F 5 "" H 12900 2950 50  0001 C CNN "Material"
 F 6 "" H 12900 2950 50  0001 C CNN "Power"
-F 7 "1%" H 12900 2950 50  0001 C CNN "Tolerance"
+F 7 "5%" H 12900 2950 50  0001 C CNN "Tolerance"
 F 8 "Vishay Dale" H 12900 2950 50  0001 C CNN "Manufacturer"
-F 9 "	CRCW06034K70JNEAC" H 12900 2950 50  0001 C CNN "PN"
+F 9 "CRCW0603100KJNEAC" H 12900 2950 50  0001 C CNN "PN"
 	1    12900 2950
 	0    1    1    0
@@
 P 13500 3300
 F 0 "R13" V 13400 3200 50  0000 L CNN
-F 1 "4.7K" V 13600 3200 50  0000 L CNN
+F 1 "100K" V 13600 3200 50  0000 L CNN
 F 2 "Resistor_SMD:R_0603_1608Metric_Pad1.05x0.95mm_HandSolder" V 13430 3300 50  0001 C CNN
 F 3 "~" H 13500 3300 50  0001 C CNN
@@
 F 5 "" H 13500 3300 50  0001 C CNN "Material"
 F 6 "" H 13500 3300 50  0001 C CNN "Power"
-F 7 "1%" H 13500 3300 50  0001 C CNN "Tolerance"
+F 7 "5 %" H 13500 3300 50  0001 C CNN "Tolerance"
 F 8 "Vishay Dale" H 13500 3300 50  0001 C CNN "Manufacturer"
-F 9 "	CRCW06034K70JNEAC" H 13500 3300 50  0001 C CNN "PN"
+F 9 "CRCW0603100KJNEAC" H 13500 3300 50  0001 C CNN "PN"
 	1    13500 3300
 	0    1    1    0
@@
 $EndComp
 $Comp
-L Audio:4833.222 IN1
+L AudioBox-rescue:4833.222-Audio IN1
 U 1 1 5F0AC88F
 P 4850 1550
@@
 $EndComp
 $Comp
-L Audio:4833.222 IN2
+L AudioBox-rescue:4833.222-Audio IN2
 U 1 1 5F0C06A2
 P 4850 2500
@@
 $EndComp
 $Comp
-L Audio:4833.222 OUT2
+L AudioBox-rescue:4833.222-Audio OUT2
 U 1 1 5F0C0B23
 P 7000 2500
@@
 $EndComp
 $Comp
-L Audio:4833.222 OUT1
+L AudioBox-rescue:4833.222-Audio OUT1
 U 1 1 5F0D324E
 P 7000 1550
@@
 P 12400 1700
 F 0 "R8" V 12300 1600 50  0000 L CNN
-F 1 "4.7K" V 12500 1600 50  0000 L CNN
+F 1 "100K" V 12500 1600 50  0000 L CNN
 F 2 "Resistor_SMD:R_0603_1608Metric_Pad1.05x0.95mm_HandSolder" V 12330 1700 50  0001 C CNN
 F 3 "~" H 12400 1700 50  0001 C CNN
@@
 F 5 "" H 12400 1700 50  0001 C CNN "Material"
 F 6 "" H 12400 1700 50  0001 C CNN "Power"
-F 7 "1%" H 12400 1700 50  0001 C CNN "Tolerance"
+F 7 "5%" H 12400 1700 50  0001 C CNN "Tolerance"
 F 8 "Vishay Dale" H 12400 1700 50  0001 C CNN "Manufacturer"
-F 9 "	CRCW06034K70JNEAC" H 12400 1700 50  0001 C CNN "PN"
+F 9 "CRCW0603100KJNEAC" H 12400 1700 50  0001 C CNN "PN"
 	1    12400 1700
 	0    1    1    0
@@
 	1650 9750 1900 9750
 $Comp
-L Regulator_Linear:LDLN030 U10
+L AudioBox-rescue:LDLN030-Regulator_Linear U10
 U 1 1 5F24D57E
 P 2200 9850
@@
 HPL
 $Comp
-L Connector:AudioJack3_SwitchT J3
+L AudioBox-rescue:AudioJack3_SwitchT-Connector J3
 U 1 1 5F42D02B
 P 8550 2100
@@
 P 11650 1450
 F 0 "R3" V 11750 1350 50  0000 L CNN
-F 1 "2.2K" V 11850 1350 50  0000 L CNN
+F 1 "100K" V 11850 1350 50  0000 L CNN
 F 2 "Resistor_SMD:R_0603_1608Metric_Pad1.05x0.95mm_HandSolder" V 11580 1450 50  0001 C CNN
 F 3 "~" H 11650 1450 50  0001 C CNN
@@
 F 5 "" H 11650 1450 50  0001 C CNN "Material"
 F 6 "" H 11650 1450 50  0001 C CNN "Power"
-F 7 "1%" H 11650 1450 50  0001 C CNN "Tolerance"
+F 7 "5" H 11650 1450 50  0001 C CNN "Tolerance"
 F 8 "Vishay Dale" H 11650 1450 50  0001 C CNN "Manufacturer"
-F 9 "CRCW06032K20FKEA" H 11650 1450 50  0001 C CNN "PN"
+F 9 "CRCW0603100KJNEAC" H 11650 1450 50  0001 C CNN "PN"
 	1    11650 1450
 	0    1    1    0
